Commit message: day7 초기 코드

File: mastering_ros_robot_description_pkg/urdf/seven_dof_arm.xacro (robot description, xacro)
@@ -115,5 +115,5 @@
   </link>
   <gazebo reference="base_link">
-    <material>Gazebo/White</material>
+    <material>Gazebo/Red</material>
   </gazebo>
   <joint name="shoulder_pan_joint" type="revolute">
@@ -144,5 +144,5 @@
   </link>
   <gazebo reference="shoulder_pan_link">
-    <material>Gazebo/Red</material>
+    <material>Gazebo/Blue</material>
   </gazebo>
   <joint name="shoulder_pitch_joint" type="revolute">
@@ -173,5 +173,5 @@
   </link>
   <gazebo reference="shoulder_pitch_link">
-    <material>Gazebo/White</material>
+    <material>Gazebo/Red</material>
   </gazebo>
   <joint name="elbow_roll_joint" type="revolute">
@@ -202,5 +202,5 @@
   </link>
   <gazebo reference="elbow_roll_link">
-    <material>Gazebo/Black</material>
+    <material>Gazebo/Yellow</material>
   </gazebo>
   <joint name="elbow_pitch_joint" type="revolute">
@@ -231,5 +231,5 @@
   </link>
   <gazebo reference="elbow_pitch_link">
-    <material>Gazebo/Red</material>
+    <material>Gazebo/Blue</material>
   </gazebo>
   <joint name="wrist_roll_joint" type="revolute">
@@ -259,5 +259,5 @@
   </link>
   <gazebo reference="wrist_roll_link">
-    <material>Gazebo/Black</material>
+    <material>Gazebo/Yellow</material>
   </gazebo>
   <joint name="wrist_pitch_joint" type="revolute">
@@ -288,5 +288,5 @@
   </link>
   <gazebo reference="wrist_pitch_link">
-    <material>Gazebo/White</material>
+    <material>Gazebo/Red</material>
   </gazebo>
   <joint name="gripper_roll_joint" type="revolute">
@@ -320,5 +320,5 @@
   </link>
   <gazebo reference="gripper_roll_link">
-    <material>Gazebo/Red</material>
+    <material>Gazebo/Blue</material>
   </gazebo>
   <joint name="finger_joint1" type="prismatic">
@@ -347,5 +347,5 @@
   </link>
   <gazebo reference="l_gripper_aft_link">
-    <material>Gazebo/White</material>
+    <material>Gazebo/Red</material>
   </gazebo>
 <!-- Joint between Wrist roll and finger 2 -->
@@ -372,5 +372,5 @@
   </link>
   <gazebo reference="r_gripper_aft_link">
-    <material>Gazebo/White</material>
+    <material>Gazebo/Red</material>
   </gazebo>
     <!-- Grasping frame -->
